Commit message: moveit,ros2_control真机全连路打通

File: src/dm_armx_config/config/DM_Armx.urdf.xacro (robot description, xacro)
@@ -6,4 +6,4 @@
     <!-- Import control_xacro -->
     <xacro:include filename="DM_Armx.ros2_control.xacro" />
-    <xacro:DM_Armx_ros2_control name="FakeSystem" initial_positions_file="$(arg initial_positions_file)"/>
+    <xacro:DM_Armx_ros2_control name="DmArmxSystem"/>
 </robot>

File: src/dm_armx_description/urdf/arm.urdf (robot description, URDF)
Before this commit: robot ReBot_Arm_DM, 10 links, 9 joints
Joints:
- joint joint2: limit lower=-3.14 upper=0 effort=27 velocity=50 -> lower=-3.14 upper=0.02 effort=27 velocity=50
- joint joint3: limit lower=-3.14 upper=0 effort=27 velocity=50 -> lower=-3.14 upper=0.02 effort=27 velocity=50

File: src/dm_armx_description/urdf/arm.xacro (robot description, xacro)
@@ -122,5 +122,5 @@
     <child link="link2" />                                           <!-- 子连杆：link2 -->
     <axis xyz="0 0 -1" />                                            <!-- 旋转轴：负 Z 轴（经父坐标系旋转后对应世界 Y） -->
-    <limit lower="-3.14" upper="0" effort="27" velocity="50" />      <!-- 限位：-π~0，力矩 27N·m，速度 50rad/s -->
+    <limit lower="-3.14" upper="0.02" effort="27" velocity="50" />    <!-- 限位：-π~0，上限留 0.02rad 余量吸收零位噪声 -->
   </joint>                                                           <!-- 关节 joint2 定义结束 -->
   <link name="link3">                                                <!-- 定义连杆：link3（第 3 轴，小臂） -->
@@ -170,5 +170,5 @@
     <child link="link3" />                                           <!-- 子连杆：link3 -->
     <axis xyz="0 0 1" />                                             <!-- 旋转轴：Z 轴 -->
-    <limit lower="-3.14" upper="0" effort="27" velocity="50" />      <!-- 限位：-π~0，力矩 27N·m，速度 50rad/s -->
+    <limit lower="-3.14" upper="0.02" effort="27" velocity="50" />    <!-- 限位：-π~0，上限留 0.02rad 余量吸收零位噪声 -->
   </joint>                                                           <!-- 关节 joint3 定义结束 -->
   <link name="link4">                                                <!-- 定义连杆：link4（第 4 轴，腕部） -->
