Commit message: 夹爪接入：力位混控驱动 + JTC 开合 + PVT 测试脚本
驱动（dm_armx_hardware）
- dm_bus：新增 send_force_pos（0x300+ID）
- dm_joint：JointConfig 增加 mode/scale/velocity_limit/力参数/软限位/fatal_on_error；
  换算带 scale；新增 set_force_pos；使能按模式补 0x300 保持帧；故障按 fatal_on_error 隔离
- 插件：read/write 按 mode 分支（力位混控多导出 effort），on_activate 给 effort 初值，
  CTRL_MODE 按期望模式校验，夹爪故障不拖垮整臂

配置
- xacro：finger_left（ID 7 / mode 4 / offset 6.560426 / scale 119.3103）；
  夹紧力默认 45 N、上限 48 N、current_per_force 0.0009（按实测重标）；
  joint1 offset 因误发 0xFE（保存零点）平移为 0.069238
- 夹爪 URDF effort 提到 50 N（JointLimiter 会用它钳 effort 命令）
- bringup：随 launch 自动起 gripper_force_controller，JTC 设置容差

测试
- src/test/pvt_motor_test.py：PVT（力位混控）单机测试，支持 --check/--scan/--set-mode/
  交互开合/--sweep/--csv/--disable；协议帧与 dm_frames.cpp 逐字节对齐

文档
- PROJECT_STATUS：2.2 参数与摩擦实测、5.5 JTC 链路验证结果、踩坑 15~20、变更记录
- 常用命令：夹爪开合/调力/失能救援命令与单位说明

真机验证：/gripper_controller 发 0.0 / 0.05 均 SUCCEEDED，行程 42.9 / 43.8 mm。

File: src/dm_armx_config/config/DM_Armx.ros2_control.xacro (robot description, xacro)
@@ -4,6 +4,6 @@
         <!-- 真机硬件插件：dm_armx_hardware/DmArmxHardwareInterface
              注意：这里只声明"插件真正会导出"的接口。
-             - 命令：只有 position（POS_VEL 模式）
-             - 状态：position + velocity
+             - 命令：六轴 position（POS_VEL）；夹爪 position + effort（力位混控）
+             - 状态：position + velocity；夹爪多一个 effort
              多声明用不到的接口（velocity/effort 命令）会让控制器以为能下发，实际没人发。 -->
         <ros2_control name="${name}" type="system">
@@ -24,5 +24,8 @@
                 <param name="motor_id">1</param>
                 <param name="direction">1</param>
-                <param name="offset">1.368925</param>
+                <!-- 2026-10-31：joint1 被误发 0xFE（"保存位置零点"）把电机零点清零，
+                     原始角 1.299496 → -0.000191。零点已写进驱动器 flash，物理姿态未变，
+                     故 offset 整体平移：1.368925 - 1.299496 + (-0.000191) = 0.069238 -->
+                <param name="offset">0.069238</param>
                 <param name="p_max">12.5</param>
                 <param name="v_max">10.0</param>
@@ -85,4 +88,38 @@
                 <param name="t_max">10.0</param>
             </joint>
+            <!-- ===== 夹爪：DM4310，力位混控（CTRL_MODE=4，0x300+ID）=====
+                 单指行程 0~0.05 m；实测闭合 +0.393874 rad、全开 -5.572786 rad
+                 ⇒ scale = (0.393874+5.572786)/0.05 = 119.3332 rad/m，direction = -1
+                 effort 单位是 N（夹紧力上限），不是电机力矩。 -->
+            <joint name="finger_left">
+                <command_interface name="position"/>
+                <command_interface name="effort"/>
+                <state_interface name="position"/>
+                <state_interface name="velocity"/>
+                <state_interface name="effort"/>
+                <param name="motor_id">7</param>
+                <param name="mode">4</param>
+                <param name="direction">-1</param>
+                <!-- 2026-10-31 重新实测：闭合 +6.560426，全开 +0.594911（绝对角漂了约 +6.17） -->
+                <param name="offset">6.560426</param>
+                <param name="scale">119.3103</param>
+                <param name="velocity_limit">0.08</param>
+                <param name="position_min">-0.002</param>
+                <param name="position_max">0.052</param>
+                <param name="p_max">12.5</param>
+                <param name="v_max">30.0</param>
+                <param name="t_max">10.0</param>
+                <!-- 2026-10-31 实测（直连电机 + JTC 全链路）：
+                     齿条阻力不是常数：闭合端静摩擦 ≈15 N，但越往开走越大
+                     （11mm→20.7N，24mm→30.0N，37mm→41.7N）。顶死在闭合端十几分钟后，
+                     30 N 已经拉不开（力恒定 +32 N 堵转），45 N 能顺利全行程。
+                     所以默认力必须给到 45 N 才有余量；上限受 URDF effort=50 约束。
+                     电流标幺按实测重标：i_des ≈ 0.0009 × F[N]（45N → 0.0405）。 -->
+                <param name="grip_force_default">45.0</param>
+                <param name="grip_force_max">48.0</param>
+                <param name="current_per_force">0.0009</param>
+                <!-- 夹爪故障只报警，不让整臂失能 -->
+                <param name="fatal_on_error">false</param>
+            </joint>
         </ros2_control>
     </xacro:macro>

File: src/dm_armx_description/urdf/arm.urdf (robot description, URDF)
Before this commit: robot ReBot_Arm_DM, 10 links, 9 joints
Joints:
- joint finger_left: limit lower=0 upper=0.05 effort=8 velocity=0.08 -> lower=-0.002 upper=0.052 effort=50 velocity=0.08
- joint finger_right: limit lower=-0.05 upper=0 effort=8 velocity=0.08 -> lower=-0.052 upper=0.002 effort=50 velocity=0.08

File: src/dm_armx_description/urdf/gripper.xacro (robot description, xacro)
@@ -82,5 +82,5 @@
     <child link="finger_left_link" />                                <!-- 子连杆：finger_left_link -->
     <axis xyz="0 1 0" />                                             <!-- 移动轴：Y 轴 -->
-    <limit lower="0" upper="0.05" effort="8" velocity="0.08" />      <!-- 限位：0~0.05m，力 8N，速度 0.08m/s -->
+    <limit lower="-0.002" upper="0.052" effort="50" velocity="0.08" />      <!-- 限位：-2~52mm（机械 0~50mm 各留 2mm 余量），力 50N，速度 0.08m/s -->
   </joint>                                                           <!-- 关节 finger_left 定义结束 -->
   <link name="finger_right_link">                                    <!-- 定义连杆：右手指 -->
@@ -125,5 +125,5 @@
     <child link="finger_right_link" />                               <!-- 子连杆：finger_right_link -->
     <axis xyz="0 1 0" />                                             <!-- 移动轴：Y 轴 -->
-    <limit lower="-0.05" upper="0" effort="8" velocity="0.08" />     <!-- 限位：-0.05~0m，力 8N，速度 0.08m/s -->
+    <limit lower="-0.052" upper="0.002" effort="50" velocity="0.08" />     <!-- 限位：-52~2mm，力 50N，速度 0.08m/s -->
     <mimic joint="finger_left" multiplier="-1" offset="0" />         <!-- 从动于 finger_left，乘数 -1 实现反向对称运动 -->
   </joint>                                                           <!-- 关节 finger_right 定义结束 -->
